File: bu/DevBoard.kicad_pcb (KiCad board)
At the start: 2 copper layers, 18.8 x 110 mm, 8 parts, among them J1 AudioJack2_Ground_Switch, J2 AudioJack2_Ground_Switch, J3 AudioJack2_Ground_Switch, J4 AudioJack2_Ground_Switch, J5 AudioJack2_Ground_Switch, J6 Eurorack_16_pin_power, J7 RJ45, J8 Conn_01x08_Female

Commit message: Started mark 2 Dev Board
Parts:
- J6: moved to B.Cu
- moved J8 47.6 mm to (55.0, 69.5)
- moved J6 1.20 mm to (62.7, 85.8)
- moved J1 0.50 mm to (55.5, 131.5)
- moved J2 0.50 mm to (64.8, 146.2)
Connections:
- J7 pad 1: +12V -> Jack1
- J7 pad 2: GND -> Jack2
- J7 pad 3: -12V -> +12V
- J7 pad 4: Jack5 -> Jack3
- J7 pad 5: Jack4 -> -12V
- J7 pad 6: Jack3 -> Jack4
- J7 pad 7: Jack2 -> GND
- J7 pad 8: Jack1 -> Jack5
Routing:
- net +12V: track 51.9 -> 36.2 mm, vias 1 -> 0
- net -12V: track 44.2 -> 29.1 mm, vias 1 -> 0
- net Jack1: track 55.0 -> 40.8 mm
- net +5V: track 88.3 -> 102.5 mm
- net Jack5: track 75.7 -> 88.3 mm
- net Jack3: track 51.9 -> 64.4 mm, vias 1 -> 0
- net Jack4: track 71.5 -> 83.5 mm, vias 1 -> 0
- net Gate: track 114.2 -> 105.4 mm
- net Jack2: track 54.9 -> 60.5 mm
- net CV: track 104.1 -> 106.1 mm
Other:
- board text added: "-12V"
- board text added: "Dev Board v1.0"
