File: bu/DevBoard_Panel.kicad_pcb (KiCad board)
At the start: 2 copper layers, 20.3 x 128.5 mm, 12 parts, among them J1 AudioJack2_Ground_Switch, J2 AudioJack2_Ground_Switch, J3 AudioJack2_Ground_Switch, J4 AudioJack2_Ground_Switch, J5 AudioJack2_Ground_Switch, J7 RJ45, J8 Conn_01x08_Female

Commit message: Started mark 2 Dev Board
Parts:
- removed J1, J2, J3, J4, J5: AudioJack2_Ground_Switch, PlayDice:THONKICONN_hole
- removed J7: RJ45, Connectors:RJ45_8
- removed J8: Conn_01x08_Female, Pin_Headers:Pin_Header_Straight_1x08_Pitch2.54mm
- added Ref**: Oval_Mounting_Hole, PlayDice:Oval_Mounting_Hole, F.Cu at (57.5, 53.0)
- added Ref**: Oval_Mounting_Hole, PlayDice:Oval_Mounting_Hole, F.Cu at (62.8, 175.5)
- ? (x5): value MountingHole_6.1mm -> Thonkiconn_Socket_6.1mm; footprint PlayDice:MountingHole_6.1mm -> Custom_Footprints:Thonkiconn_Socket_6.1mm
Routing:
- added copper zone on B.Cu, net (none)
- added copper zone on F.Cu, net (none)
- removed copper zone on B.Cu, net GND
- removed copper zone on F.Cu, net GND
Other:
- board text added: "+12v"
- board text added: "-12V"
- board text added: "Dev Board Panel v1.0"
- board text added: "Gnd"
- board text added: "J1"
- board text added: "J2"
- board text added: "J3"
- board text added: "J3 / 5V"
- board text added: "J4"
- board text added: "J4 / CV"
- board text added: "J5"
- board text added: "J5 / Gate"
- board text added: "[CV]"
- board text added: "[Gate]"
