File: DevBoard.kicad_sch (KiCad schematic)
At the start: 82 parts

Commit message: First draft of schematic done; started laying out PCB
Parts:
- added C16, C17, C19, C23: 100nF, Capacitor_SMD:C_0805_2012Metric, symbol Device:C_Small
- added C18, C22: 10uF, Capacitor_SMD:C_0805_2012Metric, symbol Device:C_Small
- added C20, C21: 2.2uF, Capacitor_SMD:C_0805_2012Metric, symbol Device:C_Small
- added C24, C25: 1nF, Capacitor_SMD:C_0805_2012Metric, symbol Device:C_Small
- added C26, C27: 100pF, Capacitor_SMD:C_0805_2012Metric, symbol Device:C_Small
- added C28, C29: 1uF, Capacitor_SMD:C_0805_2012Metric, symbol Device:C_Small
- added H1, H2, H3, H4: MountingHole, MountingHole:MountingHole_3.2mm_M3, symbol Mechanical:MountingHole
- added J18: DAC_I2S, Connector_PinHeader_2.54mm:PinHeader_1x03_P2.54mm_Vertical, symbol Connector:Conn_01x03_Pin
- added J19: DAC_OUT, Connector_PinHeader_2.54mm:PinHeader_1x02_P2.54mm_Vertical, symbol Connector:Conn_01x02_Pin
- added J20, J21: DAC_Amplified, Connector_PinHeader_2.54mm:PinHeader_1x02_P2.54mm_Vertical, symbol Connector:Conn_01x02_Pin
- added J22: Voltmeter_Power, TestPoint:TestPoint_Pad_4.0x4.0mm, symbol Connector:Conn_01x01_Pin
- added J23: Voltmeter_Positive, Connector_PinHeader_2.54mm:PinHeader_1x01_P2.54mm_Vertical, symbol Connector:Conn_01x01_Pin
- added J24: Voltmeter_Ground, TestPoint:TestPoint_Pad_4.0x4.0mm, symbol Connector:Conn_01x01_Pin
- added J25: Conn_01x05_Pin, Connector_PinHeader_2.54mm:PinHeader_1x05_P2.54mm_Vertical, symbol Connector:Conn_01x05_Pin
- added J26: Pot1, Connector_PinHeader_2.54mm:PinHeader_1x01_P2.54mm_Vertical, symbol Connector:Conn_01x01_Pin
- added J27: Pot2, Connector_PinHeader_2.54mm:PinHeader_1x01_P2.54mm_Vertical, symbol Connector:Conn_01x01_Pin
- added J28: Pot3, Connector_PinHeader_2.54mm:PinHeader_1x01_P2.54mm_Vertical, symbol Connector:Conn_01x01_Pin
- added J29: Pot4, Connector_PinHeader_2.54mm:PinHeader_1x01_P2.54mm_Vertical, symbol Connector:Conn_01x01_Pin
- added J30: CV_In, Connector_PinHeader_2.54mm:PinHeader_1x02_P2.54mm_Vertical, symbol Connector:Conn_01x02_Pin
- added J31: Audio12V_In, Connector_PinHeader_2.54mm:PinHeader_1x02_P2.54mm_Vertical, symbol Connector:Conn_01x02_Pin
- added J32: Audio_Scaled_Out, Connector_PinHeader_2.54mm:PinHeader_1x02_P2.54mm_Vertical, symbol Connector:Conn_01x02_Pin
- added J33: CV_Scaled_Out, Connector_PinHeader_2.54mm:PinHeader_1x02_P2.54mm_Vertical, symbol Connector:Conn_01x02_Pin
- added R30, R31: 2k2, Resistor_SMD:R_0805_2012Metric, symbol Device:R
- added R32, R33: 10k, Resistor_SMD:R_0805_2012Metric, symbol Device:R
- added R34, R35: 47k, Resistor_SMD:R_0805_2012Metric, symbol Device:R
- added U6: PCM5100APW, Custom_Footprints:SSOP-20_4.4x6.5mm_Pitch0.65mm_Round_Pads, symbol PCM5100APW:PCM5100APW
- added U8: TL072, Package_SO:SOIC-8_3.9x4.9mm_P1.27mm, symbol Amplifier_Operational:TL072
- C1, C2, C3, C4: renamed from C?; footprint Capacitors_SMD:C_0603_HandSoldering -> Capacitor_SMD:C_0805_2012Metric
- C10, C14, C5, C6, C7, C8, C9: renamed from C?; footprint Capacitor_SMD:C_0603_1608Metric -> Capacitor_SMD:C_0805_2012Metric
- C11, C12, C13, C15: renamed from C?; symbol Encoder:CP_Small -> Device:C_Polarized_Small
- D1, D2: renamed from D?; footprint (none) -> LED_SMD:LED_0603_1608Metric
- J1, J2, J3, J4, J5, J6, J7, J8: renamed from J?; symbol Connector:Conn_01x02_Male -> Connector:Conn_01x02_Pin
- J10, J12, J13, J14, J15, J16, J17, J9: renamed from J?; symbol Connector:Conn_01x03_Male -> Connector:Conn_01x03_Pin
- J11: renamed from J?; footprint (none) -> Custom_Footprints:RJ45_Amphenol_Style
- R1, R10, R11, R12, R2, R3, R4, R5, R6, R7, R8, R9: renamed from R?; footprint Resistors_SMD:R_0603_HandSoldering -> Resistor_SMD:R_0805_2012Metric
- R13, R14, R17, R18, R19, R20, R21, R22, R23, R24: renamed from R?; footprint Resistor_SMD:R_0603_1608Metric_Pad0.98x0.95mm_HandSolder -> Resistor_SMD:R_0805_2012Metric
- R15, R16, R25, R26, R27, R28, R29: renamed from R?; footprint Resistor_SMD:R_0603_1608Metric -> Resistor_SMD:R_0805_2012Metric
- SW1: renamed from SW?; footprint (none) -> Button_Switch_THT:SW_Push_2P2T_Toggle_CK_PVA2OAH5xxxxxxV2
- U1: renamed from U?; footprint SMD_Packages:SOIC-14_N -> Package_SO:SOIC-14_3.9x8.7mm_P1.27mm
- U3: renamed from U?; symbol Regulator_Linear:LM1117-3.3 -> Regulator_Linear:LM1117MP-3.3
- U4: renamed from U?; symbol Regulator_Linear:LM1117-5.0 -> Regulator_Linear:LM1117MP-5.0
- gave numbers to parts that had none: 7
Connections:
- net +12V: now also C28.2, J22.1 (Pin_1), U8.8 (V+)
- net +3.3VA: now also C16.1, C17.1, C18.1, U6.1 (CPVDD), U6.8 (AVDD)
- net +3V3: now also C19.1, C22.1, U6.17 (XSMT), U6.20 (DVDD)
- net -12V: now also C29.2, U8.4 (V-)
- net Audio_In1: no longer R2.2
- net Audio_In2: no longer R4.2
- net Audio_Scaled1: now also J32.1 (Pin_1)
- net Audio_Scaled2: now also J32.2 (Pin_2)
- net CV_In1: now also J30.2 (Pin_2)
- net CV_In2: now also J30.1 (Pin_1)
- net CV_Scaled1: now also J33.1 (Pin_1)
- net GND: now also C16.2, C17.2, C18.2, C19.2, C21.2, C22.2, C23.1, C24.2, C25.2, C28.1, C29.1, J24.1 (Pin_1), U6.10 (DEMP), U6.11 (FLT), U6.12 (SCK), U6.16 (FMT), U6.19 (DGND), U6.3 (CPGND), U6.9 (AGND), U8.3 (+), U8.5 (+)
- net Interconnect1: now also J25.1 (Pin_1)
- net Interconnect2: now also J25.2 (Pin_2)
- net Interconnect3: now also J25.3 (Pin_3)
- net Interconnect4_GATE: now also J25.4 (Pin_4)
- net Interconnect5_CV: now also J25.5 (Pin_5)
- net at RV4.2: now also J29.1 (Pin_1)
- net at RV1.2: now also J26.1 (Pin_1)
- net at RV2.2: now also J27.1 (Pin_1)
- net at RV3.2: now also J28.1 (Pin_1)
- net CD_Scaled2 renamed CV_Scaled2
- net CV_Scaled2: now also J33.2 (Pin_2)
- new net: C23.2, U6.18 (LDOO)
- new net: C20.1, U6.2 (CAPP)
- new net: C20.2, U6.4 (CAPM)
- new net: C21.1, U6.5 (VNEG)
- new net: C27.2, R33.1, R35.2, U8.6 (-)
- new net: C26.2, R32.1, R34.2, U8.2 (-)
- new net: C24.1, R30.1, R32.2
- new net: C25.1, R31.1, R33.2
- new net +VDC: J23.1 (Pin_1)
- new net Audio12V_In1: J31.1 (Pin_1), R2.2
- new net Audio12V_In2: J31.2 (Pin_2), R4.2
- new net DAC_BCLK: J18.3 (Pin_3), U6.13 (BCK)
- new net DAC_DATA: J18.2 (Pin_2), U6.14 (DIN)
- new net DAC_LRCLK: J18.1 (Pin_1), U6.15 (LRCK)
- new net DAC_OUT_AMP_L: C26.1, J20.1 (Pin_1), J21.1 (Pin_1), R34.1, U8.1
- new net DAC_OUT_AMP_R: C27.1, J20.2 (Pin_2), J21.2 (Pin_2), R35.1, U8.7
- new net DAC_OUT_L: J19.1 (Pin_1), R30.2, U6.6 (OUTL)
- new net DAC_OUT_R: J19.2 (Pin_2), R31.2, U6.7 (OUTR)
Other:
- note added: "Audio to MCU Scaling"
- note added: "CV to MCU Scaling"
- note added: "FLT: connect to ground for higher latency but less ringing"
- note added: "MCU to Audio Amplifiers"
- note added: "MCU to CV Amplifiers"
- note removed: "MCU Audio Amplifiers"
- note removed: "MCU CV Amplifiers"
- note removed: "MCU Input Scaling"
- moved on the sheet: C10, C3, C4, C7, C8, C9, R11, R12, R5, R6, R7, R8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

Commit message: Started PCB layout
Connections:
- net Audio12V_In2: now also J32.1 (Pin_1); no longer J31.2 (Pin_2)
- net Audio_In2: now also J3.1 (Pin_1), J4.1 (Pin_1); no longer J1.2 (Pin_2), J2.2 (Pin_2)
- net Audio_Out1: now also J1.2 (Pin_2), J2.2 (Pin_2); no longer J3.1 (Pin_1), J4.1 (Pin_1)
- net Audio_Scaled1: now also J31.2 (Pin_2); no longer J32.1 (Pin_1)
- net CV1_In: now also U2.5 (+); no longer U2.10 (+)
- net CV1_Out: now also J5.2 (Pin_2), J6.2 (Pin_2); no longer J7.1 (Pin_1), J8.1 (Pin_1)
- net CV2_In: now also J7.1 (Pin_1), J8.1 (Pin_1), U2.10 (+); no longer J5.2 (Pin_2), J6.2 (Pin_2), U2.12 (+)
- net CV_In1: now also J30.1 (Pin_1); no longer J30.2 (Pin_2)
- net CV_In2: now also J33.1 (Pin_1); no longer J30.1 (Pin_1)
- net CV_Scaled1: now also J30.2 (Pin_2); no longer J33.1 (Pin_1)
- net at R18.1, R22.2: now also U2.13 (-); no longer U2.6 (-)
- net at C6.1, R16.1: now also U2.12 (+); no longer U2.5 (+)
- net at R22.1, R26.1: now also U2.14; no longer U2.7
- net at R13.1, R19.2: now also U2.6 (-); no longer U2.9 (-)
- net at R20.1, R24.1: now also U2.8; no longer U2.14
- net at R14.1, R20.2: now also U2.9 (-); no longer U2.13 (-)
- net at R19.1, R23.1: now also U2.7; no longer U2.8
Changed lines of the file:
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@@
     (effects (font (size 1.27 1.27)) (justify right bottom))
   )
-  (label "CV2_In" (at 90.17 128.27 0) (fields_autoplaced)
+  (label "CV2_In" (at 90.17 152.4 0) (fields_autoplaced)
     (effects (font (size 1.27 1.27)) (justify left bottom))
   )
@@
     (effects (font (size 1.27 1.27)) (justify left bottom))
   )
-  (label "Audio_Out1" (at 90.17 78.74 0) (fields_autoplaced)
+  (label "Audio_Out1" (at 90.17 44.45 0) (fields_autoplaced)
     (effects (font (size 1.27 1.27)) (justify left bottom))
   )
@@
     (effects (font (size 1.27 1.27)) (justify right bottom))
   )
-  (label "Audio_In2" (at 90.17 44.45 0) (fields_autoplaced)
+  (label "Audio_In2" (at 90.17 78.74 0) (fields_autoplaced)
     (effects (font (size 1.27 1.27)) (justify left bottom))
   )
-  (label "Audio_Scaled1" (at -93.98 71.12 0) (fields_autoplaced)
+  (label "Audio_Scaled1" (at -93.98 62.23 0) (fields_autoplaced)
     (effects (font (size 1.27 1.27)) (justify left bottom))
   )
@@
     (effects (font (size 1.27 1.27)) (justify left bottom))
   )
-  (label "Audio12V_In2" (at -93.98 62.23 0) (fields_autoplaced)
+  (label "Audio12V_In2" (at -93.98 71.12 0) (fields_autoplaced)
     (effects (font (size 1.27 1.27)) (justify left bottom))
   )
-  (label "CV1_Out" (at 90.17 163.83 0) (fields_autoplaced)
+  (label "CV1_Out" (at 90.17 140.97 0) (fields_autoplaced)
     (effects (font (size 1.27 1.27)) (justify left bottom))
   )
-  (label "CV1_Out" (at 90.17 152.4 0) (fields_autoplaced)
+  (label "CV1_Out" (at 90.17 128.27 0) (fields_autoplaced)
     (effects (font (size 1.27 1.27)) (justify left bottom))
   )
@@
     (effects (font (size 1.27 1.27)) (justify left bottom))
   )
-  (label "CV_Scaled1" (at -93.98 170.18 0) (fields_autoplaced)
+  (label "CV_Scaled1" (at -93.98 152.4 0) (fields_autoplaced)
     (effects (font (size 1.27 1.27)) (justify left bottom))
   )
-  (label "CV_In2" (at -93.98 152.4 0) (fields_autoplaced)
+  (label "CV_In2" (at -93.98 170.18 0) (fields_autoplaced)
     (effects (font (size 1.27 1.27)) (justify left bottom))
   )
@@
     (effects (font (size 1.27 1.27)) (justify left bottom))
   )
-  (label "Audio_Out1" (at 90.17 67.31 0) (fields_autoplaced)
+  (label "Audio_Out1" (at 90.17 31.75 0) (fields_autoplaced)
     (effects (font (size 1.27 1.27)) (justify left bottom))
   )
@@
     (effects (font (size 1.27 1.27)) (justify left bottom))
   )
-  (label "CV2_In" (at 90.17 140.97 0) (fields_autoplaced)
+  (label "CV2_In" (at 90.17 163.83 0) (fields_autoplaced)
     (effects (font (size 1.27 1.27)) (justify left bottom))
   )
@@
     (effects (font (size 1.27 1.27)) (justify left bottom))
   )
-  (label "Audio_In2" (at 90.17 31.75 0) (fields_autoplaced)
+  (label "Audio_In2" (at 90.17 67.31 0) (fields_autoplaced)
     (effects (font (size 1.27 1.27)) (justify left bottom))
   )
@@
     )
   )
-  (symbol (lib_id "Amplifier_Operational:TL074") (at 52.07 66.04 0) (unit 2)
+  (symbol (lib_id "Amplifier_Operational:TL074") (at 52.07 66.04 0) (unit 4)
     (in_bom yes) (on_board yes) (dnp no)
     (property "Reference" "U2" (at 52.07 58.42 0)
@@
       (project "DevBoard"
         (path "/cf927a28-c7bc-4509-acea-70dea4ea1f8a"
-          (reference "U2") (unit 2)
+          (reference "U2") (unit 4)
         )
       )
@@
     )
   )
-  (symbol (lib_id "Amplifier_Operational:TL074") (at 45.72 152.4 0) (unit 4)
+  (symbol (lib_id "Amplifier_Operational:TL074") (at 45.72 152.4 0) (unit 3)
     (in_bom yes) (on_board yes) (dnp no)
     (property "Reference" "U2" (at 45.72 144.78 0)
@@
       (project "DevBoard"
         (path "/cf927a28-c7bc-4509-acea-70dea4ea1f8a"
-          (reference "U2") (unit 4)
+          (reference "U2") (unit 3)
         )
       )
@@
     )
   )
-  (symbol (lib_id "Amplifier_Operational:TL074") (at 45.72 128.27 0) (unit 3)
+  (symbol (lib_id "Amplifier_Operational:TL074") (at 45.72 128.27 0) (unit 2)
     (in_bom yes) (on_board yes) (dnp no)
     (property "Reference" "U2" (at 45.72 120.65 0)
@@
       (project "DevBoard"
         (path "/cf927a28-c7bc-4509-acea-70dea4ea1f8a"
-          (reference "U2") (unit 3)
+          (reference "U2") (unit 2)
         )
       )
@@
     )
   )
-  (symbol (lib_id "Connector:Conn_01x02_Pin") (at -99.06 152.4 0) (mirror x) (unit 1)
+  (symbol (lib_id "Connector:Conn_01x02_Pin") (at -99.06 149.86 0) (unit 1)
     (in_bom yes) (on_board yes) (dnp no)
-    (property "Reference" "J30" (at -93.98 143.51 0)
+    (property "Reference" "J30" (at -93.98 158.75 0)
       (effects (font (size 1.27 1.27)) (justify right))
     )
-    (property "Value" "CV_In" (at -93.98 146.05 0)
+    (property "Value" "CV_In" (at -93.98 156.21 0)
       (effects (font (size 1.27 1.27)) (justify right))
     )
-    (property "Footprint" "Connector_PinHeader_2.54mm:PinHeader_1x02_P2.54mm_Vertical" (at -99.06 152.4 0)
+    (property "Footprint" "Connector_PinHeader_2.54mm:PinHeader_1x02_P2.54mm_Vertical" (at -99.06 149.86 0)
       (effects (font (size 1.27 1.27)) hide)
     )
-    (property "Datasheet" "~" (at -99.06 152.4 0)
+    (property "Datasheet" "~" (at -99.06 149.86 0)
       (effects (font (size 1.27 1.27)) hide)
     )
