File: Base_Controls.kicad_pcb (KiCad board)
At the start: 2 copper layers, 18.8 x 110 mm, 8 parts, among them J1 Mult_A, J2 JackA1, J3 JackA2, J4 JackA3, J5 JackA4, J6 JackA5, J7 Eurorack_10_pin_power

Commit message: Fixed normal to ground of base unit jacks
Connections:
- J2 pad 2: GND -> unconnected-(J2-Pad2)
- J3 pad 2: GND -> unconnected-(J3-Pad2)
- J4 pad 2: GND -> unconnected-(J4-Pad2)
- J5 pad 2: GND -> unconnected-(J5-Pad2)
- J6 pad 2: GND -> unconnected-(J6-Pad2)
Changed lines of the file:
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@@
   (net 7 "+12V")
   (net 8 "GND")
+  (net 9 "unconnected-(J2-Pad2)")
+  (net 10 "unconnected-(J3-Pad2)")
+  (net 11 "unconnected-(J4-Pad2)")
+  (net 12 "unconnected-(J5-Pad2)")
+  (net 13 "unconnected-(J6-Pad2)")
   (footprint "Custom_Footprints:RJ45_Molex_42878-8506" (layer "F.Cu")
     (at 59.4 72.1)
@@
     (fp_line (start 7.9 8) (end -7.9 8)
       (stroke (width 0.1) (type solid)) (layer "F.Fab"))
-    (pad "" np_thru_hole circle (at -5.67 1.7) (size 3.65 3.65) (drill 3.33) (layers "F&B.Cu" "*.SilkS" "*.Mask"))
-    (pad "" np_thru_hole circle (at 5.76 1.7) (size 3.65 3.65) (drill 3.33) (layers "F&B.Cu" "*.SilkS" "*.Mask"))
+    (pad "" np_thru_hole circle (at -5.67 1.7) (size 3.65 3.65) (drill 3.33) (layers "F&B.Cu" "*.Mask"))
+    (pad "" np_thru_hole circle (at 5.76 1.7) (size 3.65 3.65) (drill 3.33) (layers "F&B.Cu" "*.Mask"))
     (pad "1" thru_hole rect (at -4.4 -4.65) (size 1.5 1.5) (drill 0.9) (layers "*.Cu" "*.Mask")
       (net 1 "/Interconnect1") (pintype "passive"))
@@
     (fp_circle (center 0 0) (end 1.3 0)
       (stroke (width 0.15) (type solid)) (fill none) (layer "Dwgs.User"))
+    (fp_rect (start -4.6 -6.1) (end 4.6 4.6)
+      (stroke (width 0.05) (type solid)) (fill none) (layer "F.CrtYd"))
     (pad "" np_thru_hole circle (at 0 0) (size 2.5 2.5) (drill 2.5) (layers "*.Cu" "*.Mask"))
-    (pad "1" thru_hole rect (at 0 6.48) (size 2.5 1) (drill oval 1.5 0.5) (layers "*.Cu" "*.Mask" "F.SilkS")
-      (net 8 "GND") (pintype "passive"))
-    (pad "2" thru_hole rect (at 0 3.38) (size 2.5 1) (drill oval 1.5 0.5) (layers "*.Cu" "*.Mask" "F.SilkS")
-      (net 8 "GND") (pintype "passive"))
-    (pad "3" thru_hole rect (at 0 -4.92) (size 2.5 1) (drill oval 1.5 0.5) (layers "*.Cu" "*.Mask" "F.SilkS")
+    (pad "1" thru_hole rect (at 0 6.48) (size 2.5 1) (drill oval 1.5 0.5) (layers "*.Cu" "*.Mask")
+      (net 8 "GND") (pintype "passive"))
+    (pad "2" thru_hole rect (at 0 3.38) (size 2.5 1) (drill oval 1.5 0.5) (layers "*.Cu" "*.Mask")
+      (net 9 "unconnected-(J2-Pad2)") (pintype "passive+no_connect"))
+    (pad "3" thru_hole rect (at 0 -4.92) (size 2.5 1) (drill oval 1.5 0.5) (layers "*.Cu" "*.Mask")
       (net 1 "/Interconnect1") (pintype "passive"))
     (model "${CUSTOM_3D}/PJ301M-12 Thonkiconn v0.2.stp"
@@
     (fp_circle (center 0 0) (end 1.3 0)
       (stroke (width 0.15) (type solid)) (fill none) (layer "Dwgs.User"))
+    (fp_rect (start -4.6 -6.1) (end 4.6 4.6)
+      (stroke (width 0.05) (type solid)) (fill none) (layer "F.CrtYd"))
     (pad "" np_thru_hole circle (at 0 0) (size 2.5 2.5) (drill 2.5) (layers "*.Cu" "*.Mask"))
-    (pad "1" thru_hole rect (at 0 6.48) (size 2.5 1) (drill oval 1.5 0.5) (layers "*.Cu" "*.Mask" "F.SilkS")
-      (net 8 "GND") (pintype "passive"))
-    (pad "2" thru_hole rect (at 0 3.38) (size 2.5 1) (drill oval 1.5 0.5) (layers "*.Cu" "*.Mask" "F.SilkS")
-      (net 8 "GND") (pintype "passive"))
-    (pad "3" thru_hole rect (at 0 -4.92) (size 2.5 1) (drill oval 1.5 0.5) (layers "*.Cu" "*.Mask" "F.SilkS")
+    (pad "1" thru_hole rect (at 0 6.48) (size 2.5 1) (drill oval 1.5 0.5) (layers "*.Cu" "*.Mask")
+      (net 8 "GND") (pintype "passive"))
+    (pad "2" thru_hole rect (at 0 3.38) (size 2.5 1) (drill oval 1.5 0.5) (layers "*.Cu" "*.Mask")
+      (net 13 "unconnected-(J6-Pad2)") (pintype "passive+no_connect"))
+    (pad "3" thru_hole rect (at 0 -4.92) (size 2.5 1) (drill oval 1.5 0.5) (layers "*.Cu" "*.Mask")
       (net 5 "/Interconnect5") (pintype "passive"))
     (model "${CUSTOM_3D}/PJ301M-12 Thonkiconn v0.2.stp"
@@
     (fp_circle (center 0 0) (end 1.3 0)
       (stroke (width 0.15) (type solid)) (fill none) (layer "Dwgs.User"))
+    (fp_rect (start -4.6 -6.1) (end 4.6 4.6)
+      (stroke (width 0.05) (type solid)) (fill none) (layer "F.CrtYd"))
     (pad "" np_thru_hole circle (at 0 0) (size 2.5 2.5) (drill 2.5) (layers "*.Cu" "*.Mask"))
-    (pad "1" thru_hole rect (at 0 6.48) (size 2.5 1) (drill oval 1.5 0.5) (layers "*.Cu" "*.Mask" "F.SilkS")
-      (net 8 "GND") (pintype "passive"))
-    (pad "2" thru_hole rect (at 0 3.38) (size 2.5 1) (drill oval 1.5 0.5) (layers "*.Cu" "*.Mask" "F.SilkS")
-      (net 8 "GND") (pintype "passive"))
-    (pad "3" thru_hole rect (at 0 -4.92) (size 2.5 1) (drill oval 1.5 0.5) (layers "*.Cu" "*.Mask" "F.SilkS")
+    (pad "1" thru_hole rect (at 0 6.48) (size 2.5 1) (drill oval 1.5 0.5) (layers "*.Cu" "*.Mask")
+      (net 8 "GND") (pintype "passive"))
+    (pad "2" thru_hole rect (at 0 3.38) (size 2.5 1) (drill oval 1.5 0.5) (layers "*.Cu" "*.Mask")
+      (net 12 "unconnected-(J5-Pad2)") (pintype "passive+no_connect"))
+    (pad "3" thru_hole rect (at 0 -4.92) (size 2.5 1) (drill oval 1.5 0.5) (layers "*.Cu" "*.Mask")
       (net 4 "/Interconnect4") (pintype "passive"))
     (model "${CUSTOM_3D}/PJ301M-12 Thonkiconn v0.2.stp"
@@
     (fp_circle (center 0 0) (end 1.3 0)
       (stroke (width 0.15) (type solid)) (fill none) (layer "Dwgs.User"))
+    (fp_rect (start -4.6 -6.1) (end 4.6 4.6)
+      (stroke (width 0.05) (type solid)) (fill none) (layer "F.CrtYd"))
     (pad "" np_thru_hole circle (at 0 0) (size 2.5 2.5) (drill 2.5) (layers "*.Cu" "*.Mask"))
-    (pad "1" thru_hole rect (at 0 6.48) (size 2.5 1) (drill oval 1.5 0.5) (layers "*.Cu" "*.Mask" "F.SilkS")
-      (net 8 "GND") (pintype "passive"))
-    (pad "2" thru_hole rect (at 0 3.38) (size 2.5 1) (drill oval 1.5 0.5) (layers "*.Cu" "*.Mask" "F.SilkS")
-      (net 8 "GND") (pintype "passive"))
-    (pad "3" thru_hole rect (at 0 -4.92) (size 2.5 1) (drill oval 1.5 0.5) (layers "*.Cu" "*.Mask" "F.SilkS")
+    (pad "1" thru_hole rect (at 0 6.48) (size 2.5 1) (drill oval 1.5 0.5) (layers "*.Cu" "*.Mask")
+      (net 8 "GND") (pintype "passive"))
+    (pad "2" thru_hole rect (at 0 3.38) (size 2.5 1) (drill oval 1.5 0.5) (layers "*.Cu" "*.Mask")
+      (net 11 "unconnected-(J4-Pad2)") (pintype "passive+no_connect"))
+    (pad "3" thru_hole rect (at 0 -4.92) (size 2.5 1) (drill oval 1.5 0.5) (layers "*.Cu" "*.Mask")
       (net 3 "/Interconnect3") (pintype "passive"))
     (model "${CUSTOM_3D}/PJ301M-12 Thonkiconn v0.2.stp"
@@
     (fp_circle (center 0 0) (end 1.3 0)
       (stroke (width 0.15) (type solid)) (fill none) (layer "Dwgs.User"))
+    (fp_rect (start -4.6 -6.1) (end 4.6 4.6)
+      (stroke (width 0.05) (type solid)) (fill none) (layer "F.CrtYd"))
     (pad "" np_thru_hole circle (at 0 0) (size 2.5 2.5) (drill 2.5) (layers "*.Cu" "*.Mask"))
-    (pad "1" thru_hole rect (at 0 6.48) (size 2.5 1) (drill oval 1.5 0.5) (layers "*.Cu" "*.Mask" "F.SilkS")
-      (net 8 "GND") (pintype "passive"))
-    (pad "2" thru_hole rect (at 0 3.38) (size 2.5 1) (drill oval 1.5 0.5) (layers "*.Cu" "*.Mask" "F.SilkS")
-      (net 8 "GND") (pintype "passive"))
-    (pad "3" thru_hole rect (at 0 -4.92) (size 2.5 1) (drill oval 1.5 0.5) (layers "*.Cu" "*.Mask" "F.SilkS")
+    (pad "1" thru_hole rect (at 0 6.48) (size 2.5 1) (drill oval 1.5 0.5) (layers "*.Cu" "*.Mask")
+      (net 8 "GND") (pintype "passive"))
+    (pad "2" thru_hole rect (at 0 3.38) (size 2.5 1) (drill oval 1.5 0.5) (layers "*.Cu" "*.Mask")
+      (net 10 "unconnected-(J3-Pad2)") (pintype "passive+no_connect"))
+    (pad "3" thru_hole rect (at 0 -4.92) (size 2.5 1) (drill oval 1.5 0.5) (layers "*.Cu" "*.Mask")
       (net 2 "/Interconnect2") (pintype "passive"))
     (model "${CUSTOM_3D}/PJ301M-12 Thonkiconn v0.2.stp"
